Commit message: working slam and autostart (jimmy.launch)

File: jimmy_description/urdf/jimmy.urdf.xacro (robot description, xacro)
@@ -173,5 +173,12 @@
 		<parent link="base_link" />
 		<child link="raspicam" />
-		<origin xyz="0.06 0.05 ${box_height}" />
+		<origin xyz="0.06 0.05 ${box_height}" rpy="0 0 -1.57"/>
+	</joint>
+	<link name="laser">
+	</link>
+	<joint name="base_to_laser" type="fixed">
+		<parent link="base_link"/>
+		<child link="laser"/>
+		<origin xyz="0 0 0.10" rpy="0 0 -1.57"/>
 	</joint>
 	<xacro:macro name="cube_inertial" params="origin_xyz mass width height depth">

File: jimmy_drive/cfg/map.urdf.xacro (robot description, xacro)
@@ -3,10 +3,14 @@
 	<link name="map">
 	</link>
-	<link name="tagposition_0">
-	</link>
-	<joint name="map_to_0" type="fixed">
-		<parent link="map" />
-		<child link="tagposition_0" />
-		<origin xyz="2 4 2.5" rpy="3.1416 0 0" />
-	</joint>
+	<xacro:macro name="tag" params="num xyz rpy">
+		<link name="tagposition_${num}">
+		</link>
+		<joint name="map_to_${num}" type="fixed">
+			<parent link="map" />
+			<child link="tagposition_${num}" />
+			<origin xyz="${xyz}" rpy="${rpy}" />
+		</joint>
+	</xacro:macro>
+	<xacro:tag num="0" xyz="6.7 2.8 2.5" rpy="3.1416 0 -1.57"/>
+	<xacro:tag num="1" xyz="6.7 3.8 2.5" rpy="3.1416 0 1.57"/>
 </robot>
